File: beach-ws2812.kicad_pcb (KiCad board)
At the start: 4 copper layers, 260 x 120 mm, 374 parts, among them CON101 BARREL_JACK, P101 CONN_01X03, SW101 Pushbutton, SW102 Pushbutton, U101 STM32F103C(8-B)Tx, U102 LM1117-3.3, X101 8MHz

Commit message: Fixed silk screen problems found while building first prototype.
Other:
- board text added: "2018-06-24"
- board text removed: "2018-05-27"
Changed lines of the file:
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@@
   )
   (setup
-    (last_trace_width 1)
+    (last_trace_width 0.25)
     (user_trace_width 1)
     (trace_clearance 0.2)
@@
     (tags "LED NeoPixel")
     (attr smd)
-    (fp_text reference LED240 (at 0 -3.5) (layer F.SilkS)
+    (fp_text reference LED240 (at 7 0.25) (layer F.SilkS)
       (effects (font (size 1 1) (thickness 0.15)))
     )
@@
     (tags "LED NeoPixel")
     (attr smd)
-    (fp_text reference LED328 (at 0 -3.5) (layer F.SilkS)
+    (fp_text reference LED328 (at -1.85 -3.55) (layer F.SilkS)
       (effects (font (size 1 1) (thickness 0.15)))
     )
@@
     (tags "LED NeoPixel")
     (attr smd)
-    (fp_text reference LED340 (at 0 -3.5) (layer F.SilkS)
+    (fp_text reference LED340 (at -1.9 3.8) (layer F.SilkS)
       (effects (font (size 1 1) (thickness 0.15)))
     )
@@
     (tags "capacitor 0603")
     (attr smd)
-    (fp_text reference C433 (at 0 -1.9) (layer F.SilkS)
+    (fp_text reference C433 (at 0.1 2.2) (layer F.SilkS)
       (effects (font (size 1 1) (thickness 0.15)))
     )
@@
     (tags "capacitor 0603")
     (attr smd)
-    (fp_text reference C532 (at 0 -1.9) (layer F.SilkS)
+    (fp_text reference C532 (at 0.1 1.6) (layer F.SilkS)
       (effects (font (size 1 1) (thickness 0.15)))
     )
@@
     (tags "capacitor 0603")
     (attr smd)
-    (fp_text reference C612 (at 0 -1.9 180) (layer F.SilkS)
+    (fp_text reference C612 (at -3.55 -0.05 180) (layer F.SilkS)
       (effects (font (size 1 1) (thickness 0.15)))
     )
@@
     (tags "LED NeoPixel")
     (attr smd)
-    (fp_text reference LED603 (at 0 -3.5 90) (layer F.SilkS)
+    (fp_text reference LED603 (at 4.45 -1.7 180) (layer F.SilkS)
       (effects (font (size 1 1) (thickness 0.15)))
     )
@@
     )
   )
-  (gr_text 2018-05-27 (at 38.6 111.2) (layer F.SilkS)
+  (gr_text 2018-06-24 (at 38.6 111.2) (layer F.SilkS)
     (effects (font (size 3 3) (thickness 0.3)))
   )
